Commit message: changed absolute file names to relative ones

File: models/urdf/accurate_urdf_dynamic_16505/accurate_urdf_dynamic_16505.urdf (robot description, URDF)
Before this commit: robot UR5_Table, 11 links, 10 joints
Links:
- link base_link_inertia_respondable: geometry collision mesh filename=./models/urdf/accurate_urdf_dynamic_16505/accurate_urdf_dyn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; visual mesh filename=./models/urdf/accurate_urdf_dynamic_16505/accurate_urdf_dyn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
- link forearm_link_respondable: geometry collision mesh filename=./models/urdf/accurate_urdf_dynamic_16505/accurate_urdf_dyn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; visual mesh filename=./models/urdf/accurate_urdf_dynamic_16505/accurate_urdf_dyn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
- link shoulder_link_respondable: geometry collision mesh filename=./models/urdf/accurate_urdf_dynamic_16505/accurate_urdf_dyn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; visual mesh filename=./models/urdf/accurate_urdf_dynamic_16505/accurate_urdf_dyn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
- link tool0_visual: geometry visual box size=0.000500 0.000500 0.000500; visual mesh filename=./models/urdf/accurate_urdf_dynamic_16505/accurate_urdf_dyn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
- link upper_arm_link_respondable: geometry collision mesh filename=./models/urdf/accurate_urdf_dynamic_16505/accurate_urdf_dyn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; visual mesh filename=./models/urdf/accurate_urdf_dynamic_16505/accurate_urdf_dyn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
- link wrist_1_link_respondable: geometry collision mesh filename=./models/urdf/accurate_urdf_dynamic_16505/accurate_urdf_dyn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; visual mesh filename=./models/urdf/accurate_urdf_dynamic_16505/accurate_urdf_dyn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
- link wrist_2_link_respondable: geometry collision mesh filename=./models/urdf/accurate_urdf_dynamic_16505/accurate_urdf_dyn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; visual mesh filename=./models/urdf/accurate_urdf_dynamic_16505/accurate_urdf_dyn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
- link wrist_3_link_respondable: geometry collision mesh filename=./models/urdf/accurate_urdf_dynamic_16505/accurate_urdf_dyn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; visual mesh filename=./models/urdf/accurate_urdf_dynamic_16505/accurate_urdf_dyn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

File: models/urdf/accurate_urdf_static_16505/accurate_urdf_static_16505.urdf (robot description, URDF)
Before this commit: robot UR5_Stand, 11 links, 10 joints
Links:
- link base_link_inertia_respondable: geometry collision mesh filename=file:./models/urdf/accurate_urdf_static_16505/accurate_urdf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; visual mesh filename=file:./models/urdf/accurate_urdf_static_16505/accurate_urdf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
- link forearm_link_respondable: geometry collision mesh filename=file:./models/urdf/accurate_urdf_static_16505/accurate_urdf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; visual mesh filename=file:./models/urdf/accurate_urdf_static_16505/accurate_urdf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
- link shoulder_link_respondable: geometry collision mesh filename=file:./models/urdf/accurate_urdf_static_16505/accurate_urdf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; visual mesh filename=file:./models/urdf/accurate_urdf_static_16505/accurate_urdf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
- link tool0_visual: geometry visual box size=0.000500 0.000500 0.000500; visual mesh filename=file:./models/urdf/accurate_urdf_static_16505/accurate_urdf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
- link upper_arm_link_respondable: geometry collision mesh filename=file:./models/urdf/accurate_urdf_static_16505/accurate_urdf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; visual mesh filename=file:./models/urdf/accurate_urdf_static_16505/accurate_urdf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
- link wrist_1_link_respondable: geometry collision mesh filename=file:./models/urdf/accurate_urdf_static_16505/accurate_urdf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; visual mesh filename=file:./models/urdf/accurate_urdf_static_16505/accurate_urdf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
- link wrist_2_link_respondable: geometry collision mesh filename=file:./models/urdf/accurate_urdf_static_16505/accurate_urdf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; visual mesh filename=file:./models/urdf/accurate_urdf_static_16505/accurate_urdf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
- link wrist_3_link_respondable: geometry collision mesh filename=file:./models/urdf/accurate_urdf_static_16505/accurate_urdf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; visual mesh filename=file:./models/urdf/accurate_urdf_static_16505/accurate_urdf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

File: models/urdf/ur5_static_alpha/ur5_static_alpha.urdf (robot description, URDF)
Before this commit: robot UR5_stand, 17 links, 16 joints
Links:
- link LauxLink1Visible_visual_visual_visual_visual_visual: geometry visual mesh filename=file:./models/urdf/ur5_static_alpha/ur5_static_alpha_LauxLi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; visual mesh filename=file:./models/urdf/ur5_static_alpha/ur5_static_alpha_LauxLi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
- link LauxLink2Visible_visual_visual_visual_visual_visual: geometry visual mesh filename=file:./models/urdf/ur5_static_alpha/ur5_static_alpha_LauxLi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; visual mesh filename=file:./models/urdf/ur5_static_alpha/ur5_static_alpha_LauxLi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
- link LfingerTip_respondable_respondable_respondable_respondable_respondable: geometry collision box size=0.008509 0.014223 0.025144; collision box size=0.009509 0.025404 0.036832
- link Lfinger_respondable_respondable_respondable_respondable_respondable: geometry collision box size=0.015803 0.033427 0.071444; visual mesh filename=file:./models/urdf/ur5_static_alpha/ur5_static_alpha_Lfinge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
- link RauxLink1Visible_visual_visual_visual_visual_visual: geometry visual mesh filename=file:./models/urdf/ur5_static_alpha/ur5_static_alpha_RauxLi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; visual mesh filename=file:./models/urdf/ur5_static_alpha/ur5_static_alpha_RauxLi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
- link RauxLink2Visible_visual_visual_visual_visual_visual: geometry visual mesh filename=file:./models/urdf/ur5_static_alpha/ur5_static_alpha_RauxLi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; visual mesh filename=file:./models/urdf/ur5_static_alpha/ur5_static_alpha_RauxLi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
- link RfingerTip_respondable_respondable_respondable_respondable_respondable: geometry collision box size=0.008509 0.014223 0.025144; collision box size=0.009509 0.025404 0.036832
- link Rfinger_respondable_respondable_respondable_respondable_respondable: geometry collision box size=0.015803 0.033427 0.071444; visual mesh filename=file:./models/urdf/ur5_static_alpha/ur5_static_alpha_Rfinge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
- link link_2_respondable_respondable_respondable_respondable_respondable: geometry collision mesh filename=file:./models/urdf/ur5_static_alpha/ur5_static_alpha_link_2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; collision mesh filename=file:./models/urdf/ur5_static_alpha/ur5_static_alpha_link_2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
- link link_3_respondable_respondable_respondable_respondable_respondable: geometry collision mesh filename=file:./models/urdf/ur5_static_alpha/ur5_static_alpha_link_3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; collision mesh filename=file:./models/urdf/ur5_static_alpha/ur5_static_alpha_link_3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
- link link_4_respondable_respondable_respondable_respondable_respondable: geometry collision mesh filename=file:./models/urdf/ur5_static_alpha/ur5_static_alpha_link_4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; collision mesh filename=file:./models/urdf/ur5_static_alpha/ur5_static_alpha_link_4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
- link link_5_respondable_respondable_respondable_respondable_respondable: geometry collision mesh filename=file:./models/urdf/ur5_static_alpha/ur5_static_alpha_link_5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; collision mesh filename=file:./models/urdf/ur5_static_alpha/ur5_static_alpha_link_5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
- link link_6_respondable_respondable_respondable_respondable_respondable: geometry collision cylinder length=0.025500684976578 radius=0.036602452397346; visual mesh filename=file:./models/urdf/ur5_static_alpha/ur5_static_alpha_link_6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
- link link_respondable_respondable_respondable_respondable_respondable: geometry collision mesh filename=file:./models/urdf/ur5_static_alpha/ur5_static_alpha_link_r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; collision mesh filename=file:./models/urdf/ur5_static_alpha/ur5_static_alpha_link_r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
- link robot_base: geometry collision cylinder length=0.012300089001656 radius=0.056886240839958; collision cylinder length=0.017000352963805 radius=0.072642646729946
- link robotiq_base_respondable_respondable_respondable_respondable_respondable: geometry collision box size=0.017463 0.050800 0.057938; collision box size=0.030480 0.051435 0.139700
- link static: geometry visual mesh filename=file:./models/urdf/ur5_static_alpha/ur5_static_alpha_static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

Commit message: added a function (generate_continuous_balanced_dual_arm_ik_of_trajectory) that [almost] optimally divides the work between the two arms in each interval. It runs fast (less than 5 hours on a weak laptop) and may be further accelerated as most cores are at rest.

File: models/urdf/accurate_urdf_dynamic_16505/accurate_urdf_dynamic_16505.urdf (robot description, URDF)
Before this commit: robot UR5_Table, 11 links, 10 joints
Links:
- link base_link_inertia_respondable: geometry collision mesh filename=models/urdf/accurate_urdf_dynamic_16505/accurate_urdf_dynam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; visual mesh filename=models/urdf/accurate_urdf_dynamic_16505/accurate_urdf_dynam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
- link forearm_link_respondable: geometry collision mesh filename=models/urdf/accurate_urdf_dynamic_16505/accurate_urdf_dynam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; visual mesh filename=models/urdf/accurate_urdf_dynamic_16505/accurate_urdf_dynam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
- link shoulder_link_respondable: geometry collision mesh filename=models/urdf/accurate_urdf_dynamic_16505/accurate_urdf_dynam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; visual mesh filename=models/urdf/accurate_urdf_dynamic_16505/accurate_urdf_dynam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
- link tool0_visual: geometry visual box size=0.000500 0.000500 0.000500; visual mesh filename=models/urdf/accurate_urdf_dynamic_16505/accurate_urdf_dynam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
- link upper_arm_link_respondable: geometry collision mesh filename=models/urdf/accurate_urdf_dynamic_16505/accurate_urdf_dynam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; visual mesh filename=models/urdf/accurate_urdf_dynamic_16505/accurate_urdf_dynam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
- link wrist_1_link_respondable: geometry collision mesh filename=models/urdf/accurate_urdf_dynamic_16505/accurate_urdf_dynam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; visual mesh filename=models/urdf/accurate_urdf_dynamic_16505/accurate_urdf_dynam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
- link wrist_2_link_respondable: geometry collision mesh filename=models/urdf/accurate_urdf_dynamic_16505/accurate_urdf_dynam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; visual mesh filename=models/urdf/accurate_urdf_dynamic_16505/accurate_urdf_dynam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
- link wrist_3_link_respondable: geometry collision mesh filename=models/urdf/accurate_urdf_dynamic_16505/accurate_urdf_dynam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; visual mesh filename=models/urdf/accurate_urdf_dynamic_16505/accurate_urdf_dynam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

File: models/urdf/accurate_urdf_static_16505/accurate_urdf_static_16505.urdf (robot description, URDF)
Before this commit: robot UR5_Stand, 11 links, 10 joints
Links:
- link base_link_inertia_respondable: geometry collision mesh filename=models/urdf/accurate_urdf_static_16505/accurate_urdf_static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; visual mesh filename=models/urdf/accurate_urdf_static_16505/accurate_urdf_static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
- link forearm_link_respondable: geometry collision mesh filename=models/urdf/accurate_urdf_static_16505/accurate_urdf_static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; visual mesh filename=models/urdf/accurate_urdf_static_16505/accurate_urdf_static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
- link shoulder_link_respondable: geometry collision mesh filename=models/urdf/accurate_urdf_static_16505/accurate_urdf_static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; visual mesh filename=models/urdf/accurate_urdf_static_16505/accurate_urdf_static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
- link tool0_visual: geometry visual box size=0.000500 0.000500 0.000500; visual mesh filename=models/urdf/accurate_urdf_static_16505/accurate_urdf_static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
- link upper_arm_link_respondable: geometry collision mesh filename=models/urdf/accurate_urdf_static_16505/accurate_urdf_static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; visual mesh filename=models/urdf/accurate_urdf_static_16505/accurate_urdf_static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
- link wrist_1_link_respondable: geometry collision mesh filename=models/urdf/accurate_urdf_static_16505/accurate_urdf_static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; visual mesh filename=models/urdf/accurate_urdf_static_16505/accurate_urdf_static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
- link wrist_2_link_respondable: geometry collision mesh filename=models/urdf/accurate_urdf_static_16505/accurate_urdf_static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; visual mesh filename=models/urdf/accurate_urdf_static_16505/accurate_urdf_static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
- link wrist_3_link_respondable: geometry collision mesh filename=models/urdf/accurate_urdf_static_16505/accurate_urdf_static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; visual mesh filename=models/urdf/accurate_urdf_static_16505/accurate_urdf_static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

File: models/urdf/ur5_static_alpha/ur5_static_alpha.urdf (robot description, URDF)
Before this commit: robot UR5_stand, 17 links, 16 joints
Links:
- link LauxLink1Visible_visual_visual_visual_visual_visual: geometry visual mesh filename=models/urdf/ur5_static_alpha/ur5_static_alpha_LauxLink1Visi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; visual mesh filename=models/urdf/ur5_static_alpha/ur5_static_alpha_LauxLink1Visi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
- link LauxLink2Visible_visual_visual_visual_visual_visual: geometry visual mesh filename=models/urdf/ur5_static_alpha/ur5_static_alpha_LauxLink2Visi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; visual mesh filename=models/urdf/ur5_static_alpha/ur5_static_alpha_LauxLink2Visi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
- link LfingerTip_respondable_respondable_respondable_respondable_respondable: geometry collision box size=0.008509 0.014223 0.025144; collision box size=0.009509 0.025404 0.036832
- link Lfinger_respondable_respondable_respondable_respondable_respondable: geometry collision box size=0.015803 0.033427 0.071444; visual mesh filename=models/urdf/ur5_static_alpha/ur5_static_alpha_Lfinger_respo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
- link RauxLink1Visible_visual_visual_visual_visual_visual: geometry visual mesh filename=models/urdf/ur5_static_alpha/ur5_static_alpha_RauxLink1Visi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; visual mesh filename=models/urdf/ur5_static_alpha/ur5_static_alpha_RauxLink1Visi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
- link RauxLink2Visible_visual_visual_visual_visual_visual: geometry visual mesh filename=models/urdf/ur5_static_alpha/ur5_static_alpha_RauxLink2Visi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; visual mesh filename=models/urdf/ur5_static_alpha/ur5_static_alpha_RauxLink2Visi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
- link RfingerTip_respondable_respondable_respondable_respondable_respondable: geometry collision box size=0.008509 0.014223 0.025144; collision box size=0.009509 0.025404 0.036832
- link Rfinger_respondable_respondable_respondable_respondable_respondable: geometry collision box size=0.015803 0.033427 0.071444; visual mesh filename=models/urdf/ur5_static_alpha/ur5_static_alpha_Rfinger_respo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
- link link_2_respondable_respondable_respondable_respondable_respondable: geometry collision mesh filename=models/urdf/ur5_static_alpha/ur5_static_alpha_link_2_respon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; collision mesh filename=models/urdf/ur5_static_alpha/ur5_static_alpha_link_2_respon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
- link link_3_respondable_respondable_respondable_respondable_respondable: geometry collision mesh filename=models/urdf/ur5_static_alpha/ur5_static_alpha_link_3_respon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; collision mesh filename=models/urdf/ur5_static_alpha/ur5_static_alpha_link_3_respon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
- link link_4_respondable_respondable_respondable_respondable_respondable: geometry collision mesh filename=models/urdf/ur5_static_alpha/ur5_static_alpha_link_4_respon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; collision mesh filename=models/urdf/ur5_static_alpha/ur5_static_alpha_link_4_respon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
- link link_5_respondable_respondable_respondable_respondable_respondable: geometry collision mesh filename=models/urdf/ur5_static_alpha/ur5_static_alpha_link_5_respon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; collision mesh filename=models/urdf/ur5_static_alpha/ur5_static_alpha_link_5_respon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
- link link_6_respondable_respondable_respondable_respondable_respondable: geometry collision cylinder length=0.025500684976578 radius=0.036602452397346; visual mesh filename=models/urdf/ur5_static_alpha/ur5_static_alpha_link_6_respon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
- link link_respondable_respondable_respondable_respondable_respondable: geometry collision mesh filename=models/urdf/ur5_static_alpha/ur5_static_alpha_link_responda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; collision mesh filename=models/urdf/ur5_static_alpha/ur5_static_alpha_link_responda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
- link robot_base: geometry collision cylinder length=0.012300089001656 radius=0.056886240839958; collision cylinder length=0.017000352963805 radius=0.072642646729946
- link robotiq_base_respondable_respondable_respondable_respondable_respondable: geometry collision box size=0.017463 0.050800 0.057938; collision box size=0.030480 0.051435 0.139700
- link static: geometry visual mesh filename=models/urdf/ur5_static_alpha/ur5_static_alpha_static_vis_1.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
